File: ATmega32u4/UART.kicad_sch (KiCad schematic)
At the start: 8 parts, among them U3 CH330N

Commit message: Schematic, routing and layout changes post review.
Parts:
- added R17, R18: 1k, Resistor_SMD:R_0603_1608Metric, symbol Device:R_Small
Connections:
- net RX renamed RXD
- net RXD: now also R18.1
- net TX renamed TXD
- net TXD: now also R17.1
- new net PD2-RX: R17.2
- new net PD3-TX: R18.2
Other:
- note added: "Notes: CH330N/CH340N interchangeable parts Datasheet recommends not powering CH340 and MCU separately. Could cause issues when using TX/RX port for controllers. TODO: Investigate powering separately, adding diode instead of resistors to RXD/TXD"
- note added: "RX/TX swapover here"
Changed lines of the file:
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@@
     (stroke (width 0) (type default) (color 0 0 0 0))
   )
-  (wire (pts (xy 160.02 95.25) (xy 200.66 95.25))
+  (wire (pts (xy 160.02 95.25) (xy 182.88 95.25))
     (stroke (width 0) (type default) (color 0 0 0 0))
   )
@@
     (stroke (width 0) (type default) (color 0 0 0 0))
   )
-  (wire (pts (xy 139.7 115.57) (xy 139.7 113.03))
+  (wire (pts (xy 139.7 127) (xy 139.7 113.03))
     (stroke (width 0) (type default) (color 0 0 0 0))
   )
@@
     (stroke (width 0) (type default) (color 0 0 0 0))
   )
-  (wire (pts (xy 139.7 73.66) (xy 139.7 76.2))
-    (stroke (width 0) (type default) (color 0 0 0 0))
-  )
   (wire (pts (xy 170.18 97.79) (xy 170.18 92.71))
     (stroke (width 0) (type default) (color 0 0 0 0))
@@
     (stroke (width 0) (type default) (color 0 0 0 0))
   )
+  (wire (pts (xy 139.7 63.5) (xy 139.7 76.2))
+    (stroke (width 0) (type default) (color 0 0 0 0))
+  )
   (wire (pts (xy 160.02 85.09) (xy 160.02 87.63))
     (stroke (width 0) (type default) (color 0 0 0 0))
   )
-  (wire (pts (xy 170.18 97.79) (xy 200.66 97.79))
+  (wire (pts (xy 187.96 95.25) (xy 200.66 95.25))
+    (stroke (width 0) (type default) (color 0 0 0 0))
+  )
+  (wire (pts (xy 170.18 97.79) (xy 182.88 97.79))
+    (stroke (width 0) (type default) (color 0 0 0 0))
+  )
+  (wire (pts (xy 187.96 97.79) (xy 200.66 97.79))
     (stroke (width 0) (type default) (color 0 0 0 0))
   )
@@
   (wire (pts (xy 120.65 95.25) (xy 129.54 95.25))
     (stroke (width 0) (type default) (color 0 0 0 0))
+  )
+  (text "RX/TX swapover here" (at 204.47 96.52 0)
+    (effects (font (size 1.27 1.27)) (justify left bottom))
+  )
+  (text "Notes:\n\nCH330N/CH340N interchangeable parts\n\nDatasheet recommends not powering CH340 and MCU separately. Could cause issues when using TX/RX port for controllers.\nTODO: Investigate powering separately, adding diode instead of resistors to RXD/TXD"
+    (at 12.7 196.85 0)
+    (effects (font (size 1.27 1.27)) (justify left bottom))
+  )
+  (label "TXD" (at 153.67 95.25 0)
+    (effects (font (size 1.27 1.27)) (justify left bottom))
   )
   (label "RST" (at 200.66 102.87 180)
     (effects (font (size 1.27 1.27)) (justify right bottom))
   )
-  (label "TX" (at 200.66 95.25 180)
+  (label "PD3-TX" (at 200.66 97.79 180)
     (effects (font (size 1.27 1.27)) (justify right bottom))
   )
@@
     (effects (font (size 1.27 1.27)) (justify left bottom))
   )
-  (label "RX" (at 200.66 97.79 180)
+  (label "RXD" (at 153.67 97.79 0)
+    (effects (font (size 1.27 1.27)) (justify left bottom))
+  )
+  (label "PD2-RX" (at 200.66 95.25 180)
     (effects (font (size 1.27 1.27)) (justify right bottom))
   )
@@
     (pin "2")
   )
-  (symbol (lib_id "power:GND") (at 139.7 115.57 0) (unit 1)
-    (in_bom yes) (on_board yes)
-    (property "Reference" "#PWR018" (id 0) (at 139.7 121.92 0)
-      (effects (font (size 1.27 1.27)) hide)
-    )
-    (property "Value" "GND" (id 1) (at 139.827 119.9642 0))
-    (property "Footprint" "" (id 2) (at 139.7 115.57 0)
-      (effects (font (size 1.27 1.27)) hide)
-    )
-    (property "Datasheet" "" (id 3) (at 139.7 115.57 0)
-      (effects (font (size 1.27 1.27)) hide)
-    )
-    (pin "1")
-  )
-  (symbol (lib_id "power:+5V") (at 139.7 73.66 0) (unit 1)
+  (symbol (lib_id "power:+5V") (at 139.7 63.5 0) (unit 1)
     (in_bom yes) (on_board yes) (fields_autoplaced)
-    (property "Reference" "#PWR017" (id 0) (at 139.7 77.47 0)
-      (effects (font (size 1.27 1.27)) hide)
-    )
-    (property "Value" "+5V" (id 1) (at 139.7 68.58 0))
-    (property "Footprint" "" (id 2) (at 139.7 73.66 0)
-      (effects (font (size 1.27 1.27)) hide)
-    )
-    (property "Datasheet" "" (id 3) (at 139.7 73.66 0)
+    (property "Reference" "#PWR0101" (id 0) (at 139.7 67.31 0)
+      (effects (font (size 1.27 1.27)) hide)
+    )
+    (property "Value" "+5V" (id 1) (at 139.7 58.42 0))
+    (property "Footprint" "" (id 2) (at 139.7 63.5 0)
+      (effects (font (size 1.27 1.27)) hide)
+    )
+    (property "Datasheet" "" (id 3) (at 139.7 63.5 0)
+      (effects (font (size 1.27 1.27)) hide)
+    )
+    (pin "1")
+  )
+  (symbol (lib_id "power:GND") (at 139.7 127 0) (unit 1)
+    (in_bom yes) (on_board yes)
+    (property "Reference" "#PWR018" (id 0) (at 139.7 133.35 0)
+      (effects (font (size 1.27 1.27)) hide)
+    )
+    (property "Value" "GND" (id 1) (at 139.827 131.3942 0))
+    (property "Footprint" "" (id 2) (at 139.7 127 0)
+      (effects (font (size 1.27 1.27)) hide)
+    )
+    (property "Datasheet" "" (id 3) (at 139.7 127 0)
       (effects (font (size 1.27 1.27)) hide)
     )
@@
     (pin "2")
   )
+  (symbol (lib_id "Device:R_Small") (at 185.42 95.25 90) (unit 1)
+    (in_bom yes) (on_board yes)
+    (property "Reference" "R17" (id 0) (at 182.88 93.98 90)
+      (effects (font (size 1.27 1.27)) (justify left))
+    )
+    (property "Value" "1k" (id 1) (at 187.96 93.98 90)
+      (effects (font (size 1.27 1.27)) (justify right))
+    )
+    (property "Footprint" "Resistor_SMD:R_0603_1608Metric" (id 2) (at 185.42 95.25 0)
+      (effects (font (size 1.27 1.27)) hide)
+    )
+    (property "Datasheet" "~" (id 3) (at 185.42 95.25 0)
+      (effects (font (size 1.27 1.27)) hide)
+    )
+    (pin "1")
+    (pin "2")
+  )
   (symbol (lib_id "Device:C_Small") (at 106.68 86.36 180) (unit 1)
     (in_bom yes) (on_board yes)
@@
       (effects (font (size 1.27 1.27)) hide)
     )
+    (pin "1")
+    (pin "2")
+  )
+  (symbol (lib_id "Device:R_Small") (at 185.42 97.79 90) (unit 1)
+    (in_bom yes) (on_board yes)
+    (property "Reference" "R18" (id 0) (at 182.88 99.06 90)
+      (effects (font (size 1.27 1.27)) (justify left))
+    )
+    (property "Value" "1k" (id 1) (at 187.96 99.06 90)
+      (effects (font (size 1.27 1.27)) (justify right))
+    )
+    (property "Footprint" "Resistor_SMD:R_0603_1608Metric" (id 2) (at 185.42 97.79 0)
+      (effects (font (size 1.27 1.27)) hide)
+    )
+    (property "Datasheet" "~" (id 3) (at 185.42 97.79 0)
+      (effects (font (size 1.27 1.27)) hide)
+    )

Commit message: Update notes, add io for reading cc pins, minor changes to schematic and routing.
Other:
- note removed: "Notes: CH330N/CH340N interchangeable parts Datasheet recommends not powering CH340 and MCU separately. Could cause issues when using TX/RX port for controllers. TODO: Investigate powering separately, adding diode instead of resistors to RXD/TXD"
- title: (none) -> OpenRetroPad
Changed lines of the file:
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@@
 (kicad_sch (version 20211123) (generator eeschema)
   (paper "A4")
+  (title_block
+    (title "OpenRetroPad")
+    (date "2022-12-29")
+    (rev "2")
+    (comment 3 "github.com/OpenRetroPad")
+    (comment 4 "ATmega32u4")
+  )
   (junction (at 139.7 113.03) (diameter 0) (color 0 0 0 0)
   )
@@
     (effects (font (size 1.27 1.27)) (justify left bottom))
   )
-  (text "Notes:\n\nCH330N/CH340N interchangeable parts\n\nDatasheet recommends not powering CH340 and MCU separately. Could cause issues when using TX/RX port for controllers.\nTODO: Investigate powering separately, adding diode instead of resistors to RXD/TXD"
-    (at 12.7 196.85 0)
-    (effects (font (size 1.27 1.27)) (justify left bottom))
-  )
