File: ATmega32u4/OpenRetroPad.kicad_sch (KiCad schematic)
At the start: 6 parts

Commit message: Schematic, routing and layout changes post review.
Other:
- note added: "Notes: Mounting holes are isolated, not grounded"
Changed lines of the file:
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@@
     (comment 4 "ATmega32u4")
   )
-  (bus_alias "SPI" (members "CE" "SCK" "MOSI" "MISO" "IRQ" "CSN"))
-  (bus_alias "UART" (members "TX" "RX" "RST"))
-  (bus_alias "DB25" (members "PB6" "PB5" "PF4" "PB4" "PF5" "PF6" "PD7" "PF7" "PC6" "PD4" "PD0" "PD1"))
+  (bus_alias "SPI" (members "PE6-CE" "PB1-SCK" "PB2-MOSI" "PB3-MISO" "PF1-IRQ" "PB4-CSN"))
+  (bus_alias "UART" (members "PD3-TX" "PD2-RX" "RST"))
   (bus_alias "USB" (members "DP" "DM"))
+  (bus_alias "DB25" (members "PB6" "PB5" "PF4" "PF5" "PF6" "PD7" "PF7" "PC6" "PD4" "PD0" "PD1"))
   (junction (at 127 111.76) (diameter 0) (color 0 0 0 0)
   )
@@
     (stroke (width 0) (type default) (color 0 0 0 0))
   )
+  (text "Notes:\n\nMounting holes are isolated, not grounded" (at 12.7 196.85 0)
+    (effects (font (size 1.27 1.27)) (justify left bottom))
+  )
+  (label "PB0-RX_LED" (at 111.76 156.21 0)
+    (effects (font (size 1.27 1.27)) (justify left bottom))
+  )
+  (label "PC7-LED_USER" (at 111.76 151.13 0)
+    (effects (font (size 1.27 1.27)) (justify left bottom))
+  )
   (label "PB5" (at 119.38 38.1 270)
     (effects (font (size 1.27 1.27)) (justify right bottom))
+  )
+  (label "PD5-TX_LED" (at 111.76 158.75 0)
+    (effects (font (size 1.27 1.27)) (justify left bottom))
+  )
+  (label "PE2-HWB" (at 111.76 153.67 0)
+    (effects (font (size 1.27 1.27)) (justify left bottom))
   )
   (label "RST" (at 121.92 114.3 270)
@@
       (reference "#PWR013") (unit 1) (value "GND") (footprint "")
     )
-    (path "/f64de35f-a3eb-4b10-b231-57a17c87d399/b3c80f23-acbd-425a-a520-3ce29c019169"
+    (path "/714b6847-bef8-436a-9809-c134f98f39b4/84056147-a980-4006-8250-9af655d22ae9"
       (reference "#PWR014") (unit 1) (value "+5V") (footprint "")
     )
@@
       (reference "#PWR016") (unit 1) (value "GND") (footprint "")
     )
-    (path "/e695768a-80bc-42ff-a606-2692dea2ae42/741f2427-6853-4ebb-83f8-3373005593d6"
-      (reference "#PWR017") (unit 1) (value "+5V") (footprint "")
-    )
     (path "/e695768a-80bc-42ff-a606-2692dea2ae42/53105b4c-b718-419f-be00-6911a99b80aa"
       (reference "#PWR018") (unit 1) (value "GND") (footprint "")
@@
       (reference "#PWR028") (unit 1) (value "GND") (footprint "")
     )
-    (path "/714b6847-bef8-436a-9809-c134f98f39b4/36046cf6-d707-4aea-9eb9-2034a9b5b253"
-      (reference "#PWR029") (unit 1) (value "+5V") (footprint "")
-    )
     (path "/714b6847-bef8-436a-9809-c134f98f39b4/8437b738-7bc3-4a9d-a54f-f58095bb2f7a"
       (reference "#PWR030") (unit 1) (value "+5V") (footprint "")
     )
-    (path "/714b6847-bef8-436a-9809-c134f98f39b4/cab0f48b-6a22-4b2c-add8-491676f071bc"
-      (reference "#PWR031") (unit 1) (value "GND") (footprint "")
-    )
     (path "/714b6847-bef8-436a-9809-c134f98f39b4/4320a955-fbe1-4c74-8560-dbfcbd0127a8"
       (reference "#PWR032") (unit 1) (value "GND") (footprint "")
@@
       (reference "#PWR038") (unit 1) (value "GND") (footprint "")
     )
+    (path "/e695768a-80bc-42ff-a606-2692dea2ae42/48cfd7de-c207-4b36-83ff-2b8a227ddba8"
+      (reference "#PWR0101") (unit 1) (value "+5V") (footprint "")
+    )
+    (path "/f64de35f-a3eb-4b10-b231-57a17c87d399/4f0a57e4-43fb-486e-84dd-54d0c1927a41"
+      (reference "#PWR0102") (unit 1) (value "+5V") (footprint "")
+    )
+    (path "/5c67de70-9944-4ec4-9a0d-583067d651b3/90d5c136-bddb-4cf2-af0f-64dbd6f818cd"
+      (reference "#PWR0103") (unit 1) (value "GND") (footprint "")
+    )
+    (path "/5c67de70-9944-4ec4-9a0d-583067d651b3/5775720c-0647-4905-a8b3-baebb2862c35"
+      (reference "#PWR0104") (unit 1) (value "+5V") (footprint "")
+    )
     (path "/3caf2f94-72cd-40de-b147-2caf4b503012/e347a6f3-1fbe-4eff-8dbf-d229c8539dd1"
       (reference "C1") (unit 1) (value "10u") (footprint "Capacitor_SMD:C_0805_2012Metric")
@@
       (reference "C13") (unit 1) (value "1u") (footprint "Capacitor_SMD:C_0603_1608Metric")
     )
-    (path "/f64de35f-a3eb-4b10-b231-57a17c87d399/65dfaf6f-1067-4cf4-800d-21e0d8a584d5"
-      (reference "C14") (unit 1) (value "1u") (footprint "Capacitor_SMD:C_0603_1608Metric")
-    )
     (path "/e695768a-80bc-42ff-a606-2692dea2ae42/d3d190ff-3b02-4e8a-bb65-246131453d01"
       (reference "C15") (unit 1) (value "100n") (footprint "Capacitor_SMD:C_0603_1608Metric")
@@
       (reference "C20") (unit 1) (value "100n") (footprint "Capacitor_SMD:C_0603_1608Metric")
     )
+    (path "/f64de35f-a3eb-4b10-b231-57a17c87d399/5cf5599f-081f-4e78-9385-ac6e8d37a4d9"
+      (reference "C21") (unit 1) (value "100n") (footprint "Capacitor_SMD:C_0603_1608Metric")
+    )
     (path "/3caf2f94-72cd-40de-b147-2caf4b503012/c1596543-413e-4549-acef-39889357888a"
       (reference "D1") (unit 1) (value "D_Schottky") (footprint "Diode_SMD:D_SOD-323")
@@
       (reference "D5") (unit 1) (value "1N5817") (footprint "Diode_SMD:D_SOD-323")
     )
-    (path "/714b6847-bef8-436a-9809-c134f98f39b4/0523de87-24e2-4565-b83b-3507a732cd72"
+    (path "/5c67de70-9944-4ec4-9a0d-583067d651b3/1139c864-6833-4c77-8184-5280017a4713"
       (reference "D6") (unit 1) (value "Power") (footprint "LED_SMD:LED_0603_1608Metric")
     )
@@
       (reference "J4") (unit 1) (value "DB25_Male_MountingHoles") (footprint "Connector_Dsub:DSUB-25_Male_Horizontal_P2.77x2.84mm_EdgePinOffset7.70mm_Housed_MountingHolesOffset9.12mm")
     )
-    (path "/714b6847-bef8-436a-9809-c134f98f39b4/eefb052e-71e9-4035-9346-0d1488844f6d"
+    (path "/5c67de70-9944-4ec4-9a0d-583067d651b3/999533fd-f82e-4b41-8eae-0daa63ecc4dd"
       (reference "JP1") (unit 1) (value "SJ_2_BR") (footprint "Jumper:SolderJumper-2_P1.3mm_Bridged_RoundedPad1.0x1.5mm")
     )
@@
       (reference "R12") (unit 1) (value "1k") (footprint "Resistor_SMD:R_0603_1608Metric")
     )
-    (path "/714b6847-bef8-436a-9809-c134f98f39b4/659a3901-9438-4903-a872-edc6ca23ffc6"
+    (path "/5c67de70-9944-4ec4-9a0d-583067d651b3/7da9a8cc-9fc7-4aaf-b784-578d0fd83ff5"
       (reference "R13") (unit 1) (value "1k") (footprint "Resistor_SMD:R_0603_1608Metric")
     )
@@
       (reference "R16") (unit 1) (value "330") (footprint "Resistor_SMD:R_0603_1608Metric")
     )
+    (path "/e695768a-80bc-42ff-a606-2692dea2ae42/c802af3f-6e8f-429b-9c1d-5c29c77ac3e1"
+      (reference "R17") (unit 1) (value "1k") (footprint "Resistor_SMD:R_0603_1608Metric")
+    )
+    (path "/e695768a-80bc-42ff-a606-2692dea2ae42/df3e6600-e7c2-4690-82e2-2f7ea8e9d07c"
+      (reference "R18") (unit 1) (value "1k") (footprint "Resistor_SMD:R_0603_1608Metric")
+    )
+    (path "/714b6847-bef8-436a-9809-c134f98f39b4/35267a08-f44f-42f1-b09c-1515ce6c0991"
+      (reference "R19") (unit 1) (value "10k") (footprint "Resistor_SMD:R_0603_1608Metric")
+    )
     (path "/714b6847-bef8-436a-9809-c134f98f39b4/ab1aece5-c907-4377-b211-1a641ab0362f"

Commit message: Update notes, add io for reading cc pins, minor changes to schematic and routing.
Connections:
- no-connect marks 4 -> 6
Other:
- sheet Microcontroller ports: added PB7, PD6; removed none
- sheet USB Data ports: added CC1, CC2; removed none
- sheet USB Program ports: added CC1, CC2; removed none
- note removed: "Notes: Mounting holes are isolated, not grounded"
Changed lines of the file:
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@@
   (title_block
     (title "OpenRetroPad")
-    (date "JAN-21")
-    (rev "1")
+    (date "2022-12-29")
+    (rev "2")
     (comment 3 "github.com/OpenRetroPad")
     (comment 4 "ATmega32u4")
   )
   (bus_alias "SPI" (members "PE6-CE" "PB1-SCK" "PB2-MOSI" "PB3-MISO" "PF1-IRQ" "PB4-CSN"))
+  (bus_alias "DB25" (members "PB6" "PB5" "PF4" "PF5" "PF6" "PD7" "PF7" "PC6" "PD4" "PD0" "PD1"))
   (bus_alias "UART" (members "PD3-TX" "PD2-RX" "RST"))
   (bus_alias "USB" (members "DP" "DM"))
-  (bus_alias "DB25" (members "PB6" "PB5" "PF4" "PF5" "PF6" "PD7" "PF7" "PC6" "PD4" "PD0" "PD1"))
   (junction (at 127 111.76) (diameter 0) (color 0 0 0 0)
   )
@@
   )
   (no_connect (at 274.32 60.96))
+  (no_connect (at 190.5 106.68))
   (no_connect (at 274.32 66.04))
+  (no_connect (at 190.5 109.22))
   (no_connect (at 274.32 71.12))
   (no_connect (at 274.32 55.88))
@@
     (stroke (width 0) (type default) (color 0 0 0 0))
   )
+  (wire (pts (xy 50.8 44.45) (xy 63.5 44.45))
+    (stroke (width 0) (type default) (color 0 0 0 0))
+  )
   (bus (pts (xy 139.7 40.64) (xy 127 40.64))
     (stroke (width 0) (type default) (color 0 0 0 0))
@@
     (stroke (width 0) (type default) (color 0 0 0 0))
   )
+  (wire (pts (xy 50.8 41.91) (xy 63.5 41.91))
+    (stroke (width 0) (type default) (color 0 0 0 0))
+  )
   (bus (pts (xy 121.92 35.56) (xy 139.7 35.56))
     (stroke (width 0) (type default) (color 0 0 0 0))
@@
     (stroke (width 0) (type default) (color 0 0 0 0))
   )
-  (text "Notes:\n\nMounting holes are isolated, not grounded" (at 12.7 196.85 0)
-    (effects (font (size 1.27 1.27)) (justify left bottom))
-  )
   (label "PB0-RX_LED" (at 111.76 156.21 0)
     (effects (font (size 1.27 1.27)) (justify left bottom))
   )
   (label "PC7-LED_USER" (at 111.76 151.13 0)
+    (effects (font (size 1.27 1.27)) (justify left bottom))
+  )
+  (label "PB7-CC1" (at 52.07 41.91 0)
     (effects (font (size 1.27 1.27)) (justify left bottom))
   )
@@
   (label "RST" (at 121.92 114.3 270)
     (effects (font (size 1.27 1.27)) (justify right bottom))
+  )
+  (label "PD6-CC2" (at 52.07 44.45 0)
+    (effects (font (size 1.27 1.27)) (justify left bottom))
   )
   (symbol (lib_id "Mechanical:MountingHole_Pad") (at 271.78 66.04 90) (unit 1)
@@
       (effects (font (size 1.27 1.27)) (justify left))
     )
+    (pin "CC2" output (at 190.5 109.22 180)
+      (effects (font (size 1.27 1.27)) (justify left))
+    )
+    (pin "CC1" output (at 190.5 106.68 180)
+      (effects (font (size 1.27 1.27)) (justify left))
+    )
   )
   (sheet (at 25.4 25.4) (size 25.4 25.4) (fields_autoplaced)
@@
       (effects (font (size 1.27 1.27)) (justify right))
     )
+    (pin "CC2" output (at 50.8 44.45 0)
+      (effects (font (size 1.27 1.27)) (justify right))
+    )
+    (pin "CC1" output (at 50.8 41.91 0)
+      (effects (font (size 1.27 1.27)) (justify right))
+    )
   )
   (sheet (at 25.4 127) (size 25.4 25.4) (fields_autoplaced)
@@
     (pin "{DB25}" bidirectional (at 101.6 35.56 0)
       (effects (font (size 1.27 1.27)) (justify right))
+    )
+    (pin "PB7" bidirectional (at 63.5 41.91 180)
+      (effects (font (size 1.27 1.27)) (justify left))
+    )
+    (pin "PD6" bidirectional (at 63.5 44.45 180)
+      (effects (font (size 1.27 1.27)) (justify left))
     )
   )
@@
       (reference "#FLG02") (unit 1) (value "PWR_FLAG") (footprint "")
     )
-    (path "/3caf2f94-72cd-40de-b147-2caf4b503012/c760372f-1dec-4c89-959b-7cc62ddc5ee9"
-      (reference "#FLG03") (unit 1) (value "PWR_FLAG") (footprint "")
-    )
     (path "/f64de35f-a3eb-4b10-b231-57a17c87d399/4e6b90bb-e654-425f-bab7-2ffcc4803bf9"
       (reference "#FLG04") (unit 1) (value "PWR_FLAG") (footprint "")
@@
       (reference "#FLG05") (unit 1) (value "PWR_FLAG") (footprint "")
     )
-    (path "/07c53d41-0550-42ad-9257-e12fceb2bfe2/c760372f-1dec-4c89-959b-7cc62ddc5ee9"
-      (reference "#FLG06") (unit 1) (value "PWR_FLAG") (footprint "")
+    (path "/3caf2f94-72cd-40de-b147-2caf4b503012/abbef7c2-e504-4247-b690-6a5e6faee837"
+      (reference "#FLG0101") (unit 1) (value "PWR_FLAG") (footprint "")
+    )
+    (path "/07c53d41-0550-42ad-9257-e12fceb2bfe2/abbef7c2-e504-4247-b690-6a5e6faee837"
+      (reference "#FLG0102") (unit 1) (value "PWR_FLAG") (footprint "")
     )
     (path "/3caf2f94-72cd-40de-b147-2caf4b503012/f97d72cc-95a1-42aa-83b3-3c69c70c29d1"
       (reference "#PWR01") (unit 1) (value "+5V") (footprint "")
     )
-    (path "/3caf2f94-72cd-40de-b147-2caf4b503012/41a4a14a-04d5-4b05-acf9-8fac5d2c26f0"
-      (reference "#PWR02") (unit 1) (value "GND") (footprint "")
-    )
     (path "/5c67de70-9944-4ec4-9a0d-583067d651b3/2c3fb1bd-1393-438d-a263-7d5d5f273166"
       (reference "#PWR03") (unit 1) (value "+5V") (footprint "")
@@
       (reference "#PWR06") (unit 1) (value "+5V") (footprint "")
     )
-    (path "/07c53d41-0550-42ad-9257-e12fceb2bfe2/41a4a14a-04d5-4b05-acf9-8fac5d2c26f0"
-      (reference "#PWR07") (unit 1) (value "GND") (footprint "")
-    )
     (path "/f64de35f-a3eb-4b10-b231-57a17c87d399/618bbad2-ccb5-4f99-9c84-f5310e68b759"
       (reference "#PWR08") (unit 1) (value "+5V") (footprint "")
@@
       (reference "#PWR033") (unit 1) (value "GND") (footprint "")
     )
-    (path "/3caf2f94-72cd-40de-b147-2caf4b503012/1028d9d4-8403-4788-97bc-81798d261ded"
-      (reference "#PWR034") (unit 1) (value "GND") (footprint "")
-    )
-    (path "/07c53d41-0550-42ad-9257-e12fceb2bfe2/1028d9d4-8403-4788-97bc-81798d261ded"
-      (reference "#PWR035") (unit 1) (value "GND") (footprint "")
-    )
     (path "/f64de35f-a3eb-4b10-b231-57a17c87d399/e7c005cc-8b0b-44d8-ae98-bf26182c4ef4"
       (reference "#PWR036") (unit 1) (value "+5V") (footprint "")
@@
       (reference "#PWR0104") (unit 1) (value "+5V") (footprint "")
     )
+    (path "/3caf2f94-72cd-40de-b147-2caf4b503012/1f6d1434-b97b-4809-83c6-b283eaf2dcc4"
+      (reference "#PWR0105") (unit 1) (value "GND") (footprint "")
+    )
+    (path "/07c53d41-0550-42ad-9257-e12fceb2bfe2/1f6d1434-b97b-4809-83c6-b283eaf2dcc4"
+      (reference "#PWR0106") (unit 1) (value "GND") (footprint "")
+    )
     (path "/3caf2f94-72cd-40de-b147-2caf4b503012/e347a6f3-1fbe-4eff-8dbf-d229c8539dd1"

Commit message: Change CC pin <-> ADC pin, adjust routing
Other:
- sheet Microcontroller ports: added PF0; removed PB7
Changed lines of the file:
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@@
     (effects (font (size 1.27 1.27)) (justify left bottom))
   )
-  (label "PB7-CC1" (at 52.07 41.91 0)
+  (label "PF0-CC1" (at 52.07 41.91 0)
     (effects (font (size 1.27 1.27)) (justify left bottom))
   )
@@
       (effects (font (size 1.27 1.27)) (justify right))
     )
-    (pin "PB7" bidirectional (at 63.5 41.91 180)
-      (effects (font (size 1.27 1.27)) (justify left))
-    )
     (pin "PD6" bidirectional (at 63.5 44.45 180)
       (effects (font (size 1.27 1.27)) (justify left))
     )
+    (pin "PF0" bidirectional (at 63.5 41.91 180)
+      (effects (font (size 1.27 1.27)) (justify left))
+    )
